File: HW/Resistor Panel/$Resistor Board.sch (KiCad schematic (older format))
At the start: 47 parts

Commit message: Resistor board modified: - Corrected the relays - Added the board sort circuit relay
Parts:
- R1, R10, R11, R12, R13, R14, R15, R16, R2, R20, R21, R22, R23, R24, R3, R4, R5, R6, R7, R8, R9: renamed from R?; footprint ~ -> R5
- R17, R18, R19: renamed from R?; value R -> 47K
- RLY2, RLY3, RLY4, RLY5, RLY6, RLY7, RLY8: renamed from RLY?; symbol RELAY_G6P-1114P -> RELAY_LEG-5F
- gave numbers to parts that had none: 16
Connections:
- net VCC: now also RLY2.2, RLY3.2, RLY4.2, RLY5.2, RLY6.2, RLY7.2, RLY8.2; no longer RLY2.8, RLY3.8, RLY4.8, RLY5.8, RLY6.8, RLY7.8, RLY8.8
- net at P1.3, R2.1, R4.2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: now also RLY1.3, RLY2.4; no longer RLY2.3
- net at P9.1, P9.2, P9.3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: now also RLY1.4, RLY8.3; no longer RLY8.4
- net at P3.3, R5.1, R7.2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: now also RLY2.3, RLY3.4; no longer RLY2.4, RLY3.3
- net at P4.3, R10.2, R12.2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: now also RLY3.3, RLY4.4; no longer RLY3.4, RLY4.3
- net at P5.3, R11.1, R13.2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: now also RLY4.3, RLY5.4; no longer RLY4.4, RLY5.3
- net at P6.3, R14.1, R16.2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: now also RLY5.3, RLY6.4; no longer RLY5.4, RLY6.3
- net at P7.3, R20.1, R22.2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: now also RLY6.3, RLY7.4; no longer RLY6.4, RLY7.3
- net at P10.1, P10.2, P10.3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: now also RLY7.3, RLY8.4; no longer RLY7.4, RLY8.3
