File: HW/Resistor Panel/Resistor Board.sch (KiCad schematic (older format))
At the start: 47 parts

Commit message: Resistor board modified: - Corrected the relays - Added the board sort circuit relay
Parts:
- RLY? (x8): symbol RELAY_G6P-1114P -> RELAY_LEG-5F
Connections:
- net VCC: now also RLY?.2, RLY?.2, RLY?.2, RLY?.2, RLY?.2, RLY?.2, RLY?.2, RLY?.2; no longer RLY?.8, RLY?.8, RLY?.8, RLY?.8, RLY?.8, RLY?.8, RLY?.8, RLY?.8
- net at P?.3, R?.1, R?.2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: now also RLY?.3, RLY?.5; no longer RLY?.3, RLY?.4 (x6)
- net at P?.1, P?.2, P?.3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: now also RLY?.3, RLY?.5; no longer RLY?.3, RLY?.4 (x2)

Commit message: Connector bugfix
Parts:
- R1, R10, R11, R12, R13, R14, R15, R16, R2, R20, R21, R22, R23, R24, R3, R4, R5, R6, R7, R8, R9: renamed from R?; footprint ~ -> R5
- R17, R18, R19: renamed from R?; value R -> 47K
- gave numbers to parts that had none: 23
Connections:
- net at P1.3, R2.1, R4.2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: now also RLY2.4; no longer RLY2.5
- net at P9.1, P9.2, P9.3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: now also RLY1.4; no longer RLY1.5
- net at P3.3, R5.1, R7.2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: now also RLY3.4; no longer RLY3.5
- net at P4.3, R10.2, R12.2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: now also RLY4.4; no longer RLY4.5
- net at P5.3, R11.1, R13.2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: now also RLY5.4; no longer RLY5.5
- net at P6.3, R14.1, R16.2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: now also RLY6.4; no longer RLY6.5
- net at P7.3, R20.1, R22.2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: now also RLY7.4; no longer RLY7.5
- net at P10.1, P10.2, P10.3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: now also RLY8.4; no longer RLY8.5
